File: punk75.kicad_pcb (KiCad board)
At the start: 2 copper layers, 285.8 x 124.6 mm, 192 parts, among them J1 AVR-ISP-6, SW1 RESET, SW2 BOOT, U1 ATmega32A-PU, Y1 16MHz

Commit message: added two more mounting holes and moved other two
Parts:
- added H13: M2.5, MountingHole:MountingHole_2.7mm_M2.5_ISO7380_Pad, F.Cu at (98.4, 192.1)
- added H14: M2.5, MountingHole:MountingHole_2.7mm_M2.5_ISO7380_Pad, F.Cu at (346.1, 192.1)
- moved H2 19.1 mm to (136.5, 211.1)
- moved H6 19.0 mm to (308.0, 211.2)
Routing:
- net COL7: track 294.1 -> 416.9 mm
- net COL8: track 286.6 -> 322.7 mm
- net Net-(D65-Pad2): track 153.4 -> 149.5 mm
- net Net-(D70-Pad2): track 167.5 -> 169.7 mm
- net Net-(D5-Pad2): track 88.5 -> 90.5 mm
- net COL12: track 194.7 -> 193.2 mm
- net COL6: track 332.7 -> 331.3 mm
- net COL10: track 230.9 -> 229.5 mm
- net COL9: track 274.3 -> 272.9 mm
- net COL11: track 228.0 -> 226.6 mm
- net COL13: track 190.8 -> 189.4 mm
- net COL5: track 350.4 -> 349.1 mm
