File: punk75_plate.kicad_pcb (KiCad board)
At the start: 2 copper layers, 307.8 x 146.6 mm, 8 parts

Commit message: plate now have the holes(WIP round corners)
Routing:
- added copper zone on B.Cu, net (none)
- added copper zone on F.Cu, net (none)
Changed lines of the file:
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@@
-(kicad_pcb (version 20171130) (host pcbnew "(5.1.6)-1")
+(kicad_pcb (version 20171130) (host pcbnew 5.1.6)
   (general
     (thickness 1.6)
-    (drawings 336)
+    (drawings 326)
     (tracks 0)
     (zones 0)
@@
     (41 Cmts.User user hide)
     (42 Eco1.User user hide)
-    (43 Eco2.User user hide)
+    (43 Eco2.User user)
     (44 Edge.Cuts user)
     (45 Margin user hide)
@@
       (effects (font (size 1 1) (thickness 0.15)))
     )
-    (fp_circle (center 0 0) (end 3.2 0) (layer Cmts.User) (width 0.15))
-    (fp_circle (center 0 0) (end 3.45 0) (layer F.CrtYd) (width 0.05))
+    (fp_circle (center 0 0) (end 3.45 0) (layer F.CrtYd) (width 0.05))
+    (fp_circle (center 0 0) (end 3.2 0) (layer Cmts.User) (width 0.15))
     (fp_text user %R (at 0.3 0) (layer F.Fab)
       (effects (font (size 1 1) (thickness 0.15)))
@@
       (effects (font (size 1 1) (thickness 0.15)))
     )
-    (fp_circle (center 0 0) (end 3.2 0) (layer Cmts.User) (width 0.15))
-    (fp_circle (center 0 0) (end 3.45 0) (layer F.CrtYd) (width 0.05))
+    (fp_circle (center 0 0) (end 3.45 0) (layer F.CrtYd) (width 0.05))
+    (fp_circle (center 0 0) (end 3.2 0) (layer Cmts.User) (width 0.15))
     (fp_text user %R (at 0.3 0) (layer F.Fab)
       (effects (font (size 1 1) (thickness 0.15)))
@@
       (effects (font (size 1 1) (thickness 0.15)))
     )
-    (fp_circle (center 0 0) (end 3.2 0) (layer Cmts.User) (width 0.15))
-    (fp_circle (center 0 0) (end 3.45 0) (layer F.CrtYd) (width 0.05))
+    (fp_circle (center 0 0) (end 3.45 0) (layer F.CrtYd) (width 0.05))
+    (fp_circle (center 0 0) (end 3.2 0) (layer Cmts.User) (width 0.15))
     (fp_text user %R (at 0.3 0) (layer F.Fab)
       (effects (font (size 1 1) (thickness 0.15)))
@@
       (effects (font (size 1 1) (thickness 0.15)))
     )
-    (fp_circle (center 0 0) (end 3.2 0) (layer Cmts.User) (width 0.15))
-    (fp_circle (center 0 0) (end 3.45 0) (layer F.CrtYd) (width 0.05))
+    (fp_circle (center 0 0) (end 3.45 0) (layer F.CrtYd) (width 0.05))
+    (fp_circle (center 0 0) (end 3.2 0) (layer Cmts.User) (width 0.15))
     (fp_text user %R (at 0.3 0) (layer F.Fab)
       (effects (font (size 1 1) (thickness 0.15)))
@@
       (effects (font (size 1 1) (thickness 0.15)))
     )
-    (fp_circle (center 0 0) (end 3.2 0) (layer Cmts.User) (width 0.15))
-    (fp_circle (center 0 0) (end 3.45 0) (layer F.CrtYd) (width 0.05))
+    (fp_circle (center 0 0) (end 3.45 0) (layer F.CrtYd) (width 0.05))
+    (fp_circle (center 0 0) (end 3.2 0) (layer Cmts.User) (width 0.15))
     (fp_text user %R (at 0.3 0) (layer F.Fab)
       (effects (font (size 1 1) (thickness 0.15)))
@@
       (effects (font (size 1 1) (thickness 0.15)))
     )
-    (fp_circle (center 0 0) (end 3.2 0) (layer Cmts.User) (width 0.15))
-    (fp_circle (center 0 0) (end 3.45 0) (layer F.CrtYd) (width 0.05))
+    (fp_circle (center 0 0) (end 3.45 0) (layer F.CrtYd) (width 0.05))
+    (fp_circle (center 0 0) (end 3.2 0) (layer Cmts.User) (width 0.15))
     (fp_text user %R (at 0.3 0) (layer F.Fab)
       (effects (font (size 1 1) (thickness 0.15)))
@@
       (effects (font (size 1 1) (thickness 0.15)))
     )
-    (fp_circle (center 0 0) (end 3.2 0) (layer Cmts.User) (width 0.15))
-    (fp_circle (center 0 0) (end 3.45 0) (layer F.CrtYd) (width 0.05))
+    (fp_circle (center 0 0) (end 3.45 0) (layer F.CrtYd) (width 0.05))
+    (fp_circle (center 0 0) (end 3.2 0) (layer Cmts.User) (width 0.15))
     (fp_text user %R (at 0.3 0) (layer F.Fab)
       (effects (font (size 1 1) (thickness 0.15)))
@@
       (effects (font (size 1 1) (thickness 0.15)))
     )
-    (fp_circle (center 0 0) (end 3.2 0) (layer Cmts.User) (width 0.15))
-    (fp_circle (center 0 0) (end 3.45 0) (layer F.CrtYd) (width 0.05))
+    (fp_circle (center 0 0) (end 3.45 0) (layer F.CrtYd) (width 0.05))
+    (fp_circle (center 0 0) (end 3.2 0) (layer Cmts.User) (width 0.15))
     (fp_text user %R (at 0.3 0) (layer F.Fab)
       (effects (font (size 1 1) (thickness 0.15)))
@@
   (gr_circle (center 272.74875 236.1175) (end 275.29875 236.1175) (layer Edge.Cuts) (width 0.2))
   (gr_circle (center 91.76125 236.1175) (end 94.31125 236.1175) (layer Edge.Cuts) (width 0.2))
-  (gr_line (start 68.38 109.4675) (end 68.38 227.73625) (layer Edge.Cuts) (width 0.2))
-  (gr_line (start 81.76125 241.1175) (end 362.74875 241.1175) (layer Edge.Cuts) (width 0.2))
-  (gr_line (start 376.13 227.73625) (end 376.13 107.88) (layer Edge.Cuts) (width 0.2))
   (gr_arc (start 362.74875 107.88) (end 366.13 107.88) (angle -90) (layer Edge.Cuts) (width 0.2))
   (gr_circle (center 272.74875 99.49875) (end 275.29875 99.49875) (layer Edge.Cuts) (width 0.2))
-  (gr_arc (start 81.76125 227.73625) (end 68.38 227.73625) (angle -90) (layer Edge.Cuts) (width 0.2))
-  (gr_arc (start 362.74875 107.88) (end 376.13 107.88) (angle -90) (layer Edge.Cuts) (width 0.2))
   (gr_arc (start 81.76125 107.88) (end 81.76125 104.498749) (angle -90) (layer Edge.Cuts) (width 0.2))
-  (gr_arc (start 81.76125 107.88) (end 81.76125 94.49875) (angle -90) (layer Edge.Cuts) (width 0.2))
   (gr_circle (center 91.76125 99.49875) (end 94.31125 99.49875) (layer Edge.Cuts) (width 0.2))
-  (gr_line (start 82.555 94.49875) (end 81.76125 94.49875) (layer Edge.Cuts) (width 0.2))
-  (gr_line (start 362.74875 94.49875) (end 82.555 94.49875) (layer Edge.Cuts) (width 0.2))
   (gr_circle (center 171.76125 99.49875) (end 174.311249 99.49875) (layer Edge.Cuts) (width 0.2))
   (gr_circle (center 352.74875 99.49875) (end 355.29875 99.49875) (layer Edge.Cuts) (width 0.2))
-  (gr_arc (start 362.74875 227.73625) (end 362.74875 241.1175) (angle -90) (layer Edge.Cuts) (width 0.2))
-  (gr_line (start 68.38 107.88) (end 68.38 109.4675) (layer Edge.Cuts) (width 0.2))
   (gr_line (start 376.13 227.73525) (end 376.13 107.879) (layer Edge.Cuts) (width 0.2))
   (gr_arc (start 362.74875 227.73525) (end 362.74875 241.1165) (angle -90) (layer Edge.Cuts) (width 0.2))
@@
     (effects (font (size 2 2) (thickness 0.15)) (justify mirror))
   )
+  (zone (net 0) (net_name "") (layer F.Cu) (hatch edge 0.508)
+    (connect_pads (clearance 0.508))
+    (min_thickness 0.254)
+    (fill yes (arc_segments 32) (thermal_gap 0.508) (thermal_bridge_width 0.508))
+    (polygon
+      (pts
+        (xy 383.794 248.412) (xy 49.911 251.841) (xy 49.403 82.423) (xy 382.778 82.169)
+      )
+    )
+  )
+  (zone (net 0) (net_name "") (layer B.Cu) (hatch edge 0.508)
+    (connect_pads (clearance 0.508))
+    (min_thickness 0.254)
+    (fill yes (arc_segments 32) (thermal_gap 0.508) (thermal_bridge_width 0.508))
+    (polygon
+      (pts
+        (xy 383.667 249.428) (xy 49.784 251.714) (xy 50.038 83.312) (xy 383.032 82.296)
+      )
+    )
+  )
 )

Commit message: pcb plate
Other:
- outline, holes or cut-outs redrawn
