File: punk75_plate.kicad_pcb (KiCad board)
At the start: 2 copper layers, 307.8 x 146.6 mm, 8 parts

Commit message: plate change made in the pcb
Other:
- outline, holes or cut-outs redrawn

Commit message: fixed plate and inner holes
Parts:
- REF** (x8): value M3 -> M5; footprint MountingHole:MountingHole_3.2mm_M3_Pad -> MountingHole:MountingHole_5.3mm_M5_ISO14580_Pad
Other:
- outline, holes or cut-outs redrawn
